File: kicad_main/cemicro-mp.kicad_sch (KiCad schematic)
At the start: 14 parts, among them U1 68HC11, U3 2764, U6 AMS1117-5.0

Commit message: KiCad update
Parts:
- added J1: PSU, symbol Connector_Generic:Conn_01x05
Connections:
- net +5V: no longer C1.1, C2.1, C3.1, R10.2, R11.2, R12.2, R13.2, R14.2, R15.2, R16.2, R9.2, U3.1 (VPP), U3.27 (~{PGM}), U3.28 (VCC)
- net GND: now also J1.5 (Pin_5)
- net PROG_EN: now reaches U1.2 (OC2/PA6)
- net PROG_EN: now also J1.2 (Pin_2)
- net at U1.5 (OC5/PA3): now also U3.27 (~{PGM})
- new net +13V: J1.1 (Pin_1)
- new net VCC: C1.1, C2.1, C3.1, J1.4 (Pin_4), R10.2, R11.2, R12.2, R13.2, R14.2, R15.2, R16.2, R9.2, U3.28 (VCC)
- new net VPP: J1.3 (Pin_3), U3.1 (VPP)
Other:
- title: CEMICRO Final Project Part I -> CEMICRO Final Project
- moved on the sheet: U1, U3
